File: myboard.sch (KiCad schematic (older format))
At the start: 49 parts, among them K0 KEYSW, K1 KEYSW, K10 KEYSW, K11 KEYSW, K12 KEYSW, K13 KEYSW, K2 KEYSW, K20 KEYSW, K21 KEYSW, K22 KEYSW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

Commit message: hoge
Parts:
- removed J_PRO_MICRO1: CONN_02X12, Pin_Headers:Pin_Header_Straight_2x12_Pitch1.27mm, symbol CONN_02X12
- added J1: SUPP24, keebs:Pro_Micro, symbol SUPP24
Connections:
- net col0: now also J1.20
- net col1: now also J1.19
- net col2: now also J1.18
- net col3: now also J1.17
- net row0: now also J1.16
- net row1: now also J1.15
- net row2: now also J1.14
- net row3: now also J1.13
- net row4: now also J1.5
- net row5: now also J1.6
Changed lines of the file:
@@
 LIBS:valves
 LIBS:keyboard_parts
+LIBS:myboard-cache
 EELAYER 25 0
 EELAYER END
@@
 Comment4 ""
 $EndDescr
-$Comp
-L CONN_02X12 J_PRO_MICRO1
-U 1 1 58EF57A6
-P 4050 1950
-F 0 "J_PRO_MICRO1" H 4050 2600 50  0000 C CNN
-F 1 "CONN_02X12" V 4050 1950 50  0000 C CNN
-F 2 "Pin_Headers:Pin_Header_Straight_2x12_Pitch1.27mm" H 4050 750 50  0001 C CNN
-F 3 "" H 4050 750 50  0001 C CNN
-	1    4050 1950
-	1    0    0    -1
-$EndComp
 $Comp
 L KEYSW K0
@@
 Text Label 5600 6150 1    60   ~ 0
 row5
-Text Label 4300 1800 0    60   ~ 0
+Text Label 3250 1900 0    60   ~ 0
+col1
+Text Label 3250 2000 0    60   ~ 0
+col2
+Text Label 3250 2100 0    60   ~ 0
+col3
+Text Label 3250 2200 0    60   ~ 0
+row0
+Text Label 3250 2300 0    60   ~ 0
+row1
+Text Label 3250 2400 0    60   ~ 0
+row2
+Text Label 3250 2500 0    60   ~ 0
+row3
+Text Label 2050 1800 2    60   ~ 0
+row4
+Text Label 2050 1900 2    60   ~ 0
+row5
+$Comp
+L SUPP24 J1
+U 1 1 58F37EFF
+P 2650 1950
+F 0 "J1" H 2650 2050 50  0000 C CNN
+F 1 "SUPP24" H 2650 1850 50  0000 C CNN
+F 2 "keebs:Pro_Micro" H 2650 1950 50  0001 C CNN
+F 3 "" H 2650 1950 50  0001 C CNN
+	1    2650 1950
+	1    0    0    -1
+$EndComp
+Text Label 3250 1800 0    60   ~ 0
 col0
-Text Label 4300 1900 0    60   ~ 0
-col1
-Text Label 4300 2000 0    60   ~ 0
-col2
-Text Label 4300 2100 0    60   ~ 0
-col3
-Text Label 4300 2200 0    60   ~ 0
-row0
-Text Label 4300 2300 0    60   ~ 0
-row1
-Text Label 4300 2400 0    60   ~ 0
-row2
-Text Label 4300 2500 0    60   ~ 0
-row3
-Text Label 3800 1800 2    60   ~ 0
-row4
-Text Label 3800 1900 2    60   ~ 0
-row5
 $EndSCHEMATC
